File: KICAD/pcb_capteur_graphite_V2/pcb_capteur_graphite_V2.kicad_pcb (KiCad board)
At the start: 2 copper layers, 68.6 x 53.3 mm, 8 parts, among them J1 Power, J2 Digital/PWM, J3 Analog, J4 Digital/PWM

Commit message: Progression KICAD
Parts:
- added C1: C, Capacitor_THT:C_Disc_D3.0mm_W1.6mm_P2.50mm, F.Cu at (138.5, 88.3)
- added C2: C, Capacitor_THT:C_Disc_D3.0mm_W1.6mm_P2.50mm, F.Cu at (130.8, 85.5)
- added C3: C, Capacitor_THT:C_Rect_L7.0mm_W4.5mm_P5.00mm, F.Cu at (141.8, 86.8)
- added C4: C, Capacitor_THT:C_Disc_D3.0mm_W1.6mm_P2.50mm, F.Cu at (145.8, 91.9)
- added R1: R, Resistor_THT:R_Axial_DIN0204_L3.6mm_D1.6mm_P1.90mm_Vertical, F.Cu at (137.8, 77.9)
- added R2: R, Resistor_THT:R_Axial_DIN0204_L3.6mm_D1.6mm_P1.90mm_Vertical, F.Cu at (132.3, 80.1)
- added R3: R, Resistor_THT:R_Axial_DIN0204_L3.6mm_D1.6mm_P1.90mm_Vertical, F.Cu at (135.9, 85.5)
- added R4: R, Resistor_THT:R_Axial_DIN0204_L3.6mm_D1.6mm_P1.90mm_Vertical, F.Cu at (141.5, 81.7)
- added R5: R, Resistor_THT:R_Axial_DIN0204_L3.6mm_D1.6mm_P1.90mm_Vertical, F.Cu at (150.5, 91.1)
- added U1: Blutooth_HC06, New_footprints:Bluetooth, F.Cu at (120.3, 56.8)
- added U2: LTC1050, Package_DIP:DIP-8_W7.62mm, F.Cu at (118.3, 70.7)
- added U3: capteur, New_footprints:capteur, F.Cu at (133.8, 73.5)
- added U4: oled, New_footprints:OLED, F.Cu at (159.7, 69.6)
Connections:
- J2 pad 7: /*11 -> /*11/RX
- J2 pad 8: /*10 -> /*10/TX
