File: KICAD/pcb_capteur_graphite_V2/pcb_capteur_graphite_V2.kicad_pcb (KiCad board)
At the start: 2 copper layers, 68.6 x 53.3 mm, 21 parts, among them J1 Power, J2 Digital/PWM, J3 Analog, J4 Digital/PWM, U1 Blutooth_HC06, U2 LTC1050, U3 capteur, U4 oled

Commit message: qq modification
Parts:
- moved U4 29.2 mm to (130.5, 69.5)
- moved U1 22.4 mm to (138.2, 70.2), turned to 90 degrees
Connections:
- R1 pad 1: Net-(R1-Pad1) -> Net-(U3-Pad1)
- U2 pad 2: (no net) -> Net-(C1-Pad1)
- U2 pad 3: (no net) -> Net-(C1-Pad1)
- U2 pad 4: (no net) -> GND
- U2 pad 6: (no net) -> Net-(C3-Pad2)
- U2 pad 7: (no net) -> +5V
- U3 pad 1: (no net) -> Net-(U3-Pad1)
Changed lines of the file:
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@@
   (net 28 "/*11{slash}RX")
   (net 29 "/*10{slash}TX")
-  (net 30 "Net-(R1-Pad1)")
+  (net 30 "Net-(U3-Pad1)")
   (net 31 "Net-(C3-Pad2)")
   (net 32 "/A5")
@@
     (fp_circle (center 0 0) (end 0.8 0) (layer "F.Fab") (width 0.1) (fill none))
     (pad "1" thru_hole circle (at 0 0 270) (size 1.4 1.4) (drill 0.7) (layers *.Cu *.Mask)
-      (net 30 "Net-(R1-Pad1)") (pintype "passive"))
+      (net 30 "Net-(U3-Pad1)") (pintype "passive"))
     (pad "2" thru_hole oval (at 1.9 0 270) (size 1.4 1.4) (drill 0.7) (layers *.Cu *.Mask)
       (net 16 "Net-(C1-Pad1)") (pintype "passive"))
@@
       (effects (font (size 1 1) (thickness 0.15)))
     )
-    (pad "1" thru_hole circle (at 15.24 -5.08) (size 2 2) (drill 0.8) (layers *.Cu *.Mask))
-    (pad "1" thru_hole circle (at 12.7 -5.08) (size 2 2) (drill 0.8) (layers *.Cu *.Mask))
+    (pad "1" thru_hole circle (at 15.24 -5.08) (size 2 2) (drill 0.8) (layers *.Cu *.Mask)
+      (net 30 "Net-(U3-Pad1)") (pinfunction "OUT") (pintype "bidirectional"))
+    (pad "1" thru_hole circle (at 12.7 -5.08) (size 2 2) (drill 0.8) (layers *.Cu *.Mask)
+      (net 30 "Net-(U3-Pad1)") (pinfunction "OUT") (pintype "bidirectional"))
   )
   (footprint "New_footprints:Bluetooth" (layer "F.Cu")
-    (at 120.288 56.788)
-    (property "Sheetfile" "pcb_capteur_graphite_V2.kicad_sch")
-    (property "Sheetname" "")
-    (attr through_hole)
-    (fp_text reference "U1" (at 0 -0.5 unlocked) (layer "F.SilkS")
-      (effects (font (size 1 1) (thickness 0.15)))
-    )
-    (fp_text value "Blutooth_HC06" (at 0 1 unlocked) (layer "F.Fab")
-      (effects (font (size 1 1) (thickness 0.15)))
-    )
-    (fp_text user "GND" (at 10.16 4.318 unlocked) (layer "F.SilkS")
+    (at 138.195 70.187 90)
+    (property "Sheetfile" "pcb_capteur_graphite_V2.kicad_sch")
+    (property "Sheetname" "")
+    (attr through_hole)
+    (fp_text reference "U1" (at 0 -0.5 90 unlocked) (layer "F.SilkS")
+      (effects (font (size 1 1) (thickness 0.15)))
+    )
+    (fp_text value "Blutooth_HC06" (at 0 1 90 unlocked) (layer "F.Fab")
+      (effects (font (size 1 1) (thickness 0.15)))
+    )
+    (fp_text user "GND" (at 10.16 4.318 90 unlocked) (layer "F.SilkS")
       (effects (font (size 0.8 0.8) (thickness 0.1)))
     )
-    (fp_text user "RX" (at 15.24 4.318 unlocked) (layer "F.SilkS")
+    (fp_text user "RX" (at 15.24 4.318 90 unlocked) (layer "F.SilkS")
       (effects (font (size 0.8 0.8) (thickness 0.1)))
     )
-    (fp_text user "TX" (at 12.7 4.318 unlocked) (layer "F.SilkS")
+    (fp_text user "TX" (at 12.7 4.318 90 unlocked) (layer "F.SilkS")
       (effects (font (size 0.8 0.8) (thickness 0.1)))
     )
-    (fp_text user "VCC" (at 7.62 4.318 unlocked) (layer "F.SilkS")
+    (fp_text user "VCC" (at 7.62 4.318 90 unlocked) (layer "F.SilkS")
       (effects (font (size 0.8 0.8) (thickness 0.1)))
     )
-    (fp_text user "${REFERENCE}" (at 0 2.5 unlocked) (layer "F.Fab")
+    (fp_text user "${REFERENCE}" (at 0 2.5 90 unlocked) (layer "F.Fab")
       (effects (font (size 1 1) (thickness 0.15)))
     )
     (fp_rect (start 6.096 1.27) (end 16.764 5.08) (layer "F.SilkS") (width 0.12) (fill none))
-    (pad "1" thru_hole circle (at 7.62 2.54) (size 2 2) (drill 0.8) (layers *.Cu *.Mask)
+    (pad "1" thru_hole circle (at 7.62 2.54 90) (size 2 2) (drill 0.8) (layers *.Cu *.Mask)
       (net 26 "VCC") (pinfunction "VCC") (pintype "bidirectional"))
-    (pad "2" thru_hole circle (at 10.16 2.54) (size 2 2) (drill 0.8) (layers *.Cu *.Mask)
+    (pad "2" thru_hole circle (at 10.16 2.54 90) (size 2 2) (drill 0.8) (layers *.Cu *.Mask)
       (net 1 "GND") (pinfunction "GND") (pintype "bidirectional"))
-    (pad "3" thru_hole circle (at 12.7 2.54) (size 2 2) (drill 0.8) (layers *.Cu *.Mask)
+    (pad "3" thru_hole circle (at 12.7 2.54 90) (size 2 2) (drill 0.8) (layers *.Cu *.Mask)
       (net 29 "/*10{slash}TX") (pinfunction "TX") (pintype "bidirectional"))
-    (pad "4" thru_hole circle (at 15.24 2.54) (size 2 2) (drill 0.8) (layers *.Cu *.Mask)
+    (pad "4" thru_hole circle (at 15.24 2.54 90) (size 2 2) (drill 0.8) (layers *.Cu *.Mask)
       (net 28 "/*11{slash}RX") (pinfunction "RX") (pintype "bidirectional"))
   )
@@
     (fp_line (start 6.985 8.89) (end 0.635 8.89) (layer "F.Fab") (width 0.1))
     (pad "1" thru_hole rect (at 0 0) (size 1.6 1.6) (drill 0.8) (layers *.Cu *.Mask))
-    (pad "2" thru_hole oval (at 0 2.54) (size 1.6 1.6) (drill 0.8) (layers *.Cu *.Mask))
-    (pad "3" thru_hole oval (at 0 5.08) (size 1.6 1.6) (drill 0.8) (layers *.Cu *.Mask))
-    (pad "4" thru_hole oval (at 0 7.62) (size 1.6 1.6) (drill 0.8) (layers *.Cu *.Mask))
+    (pad "2" thru_hole oval (at 0 2.54) (size 1.6 1.6) (drill 0.8) (layers *.Cu *.Mask)
+      (net 16 "Net-(C1-Pad1)") (pinfunction "IN-") (pintype "input"))
+    (pad "3" thru_hole oval (at 0 5.08) (size 1.6 1.6) (drill 0.8) (layers *.Cu *.Mask)
+      (net 16 "Net-(C1-Pad1)") (pinfunction "IN+") (pintype "input"))
+    (pad "4" thru_hole oval (at 0 7.62) (size 1.6 1.6) (drill 0.8) (layers *.Cu *.Mask)
+      (net 1 "GND") (pinfunction "V-") (pintype "input"))
     (pad "5" thru_hole oval (at 7.62 7.62) (size 1.6 1.6) (drill 0.8) (layers *.Cu *.Mask))
-    (pad "6" thru_hole oval (at 7.62 5.08) (size 1.6 1.6) (drill 0.8) (layers *.Cu *.Mask))
-    (pad "7" thru_hole oval (at 7.62 2.54) (size 1.6 1.6) (drill 0.8) (layers *.Cu *.Mask))
+    (pad "6" thru_hole oval (at 7.62 5.08) (size 1.6 1.6) (drill 0.8) (layers *.Cu *.Mask)
+      (net 31 "Net-(C3-Pad2)") (pinfunction "OUT") (pintype "output"))
+    (pad "7" thru_hole oval (at 7.62 2.54) (size 1.6 1.6) (drill 0.8) (layers *.Cu *.Mask)
+      (net 3 "+5V") (pinfunction "V+") (pintype "input"))
     (pad "8" thru_hole oval (at 7.62 0) (size 1.6 1.6) (drill 0.8) (layers *.Cu *.Mask))
     (model "${KICAD6_3DMODEL_DIR}/Package_DIP.3dshapes/DIP-8_W7.62mm.wrl"
@@
   )
   (footprint "New_footprints:OLED" (layer "F.Cu")
-    (at 159.722 69.552 90)
-    (property "Sheetfile" "pcb_capteur_graphite_V2.kicad_sch")
-    (property "Sheetname" "")
+    (at 130.48 69.52 90)
+    (property "Sheetfile" "pcb_capteur_graphite_V2.kicad_sch")
+    (property "Sheetname" "")

Commit message: le projet V2 le plus nouvelle dans session de yin, j'espere c'est le version qu'on a envoye au cathy
Parts:
- C1, C2, C4: footprint Capacitor_THT:C_Disc_D3.0mm_W1.6mm_P2.50mm -> New_footprints:Conductance
- R1, R2, R3, R4, R5: footprint Resistor_THT:R_Axial_DIN0204_L3.6mm_D1.6mm_P1.90mm_Vertical -> New_footprints:Resistor
- U4: moved to B.Cu
- moved U4 33.2 mm to (161.0, 82.7), turned to 0 degrees
- moved C1 25.3 mm to (114.8, 79.4), turned to 90 degrees
- moved R1 24.6 mm to (113.8, 72.6)
- moved C3 21.1 mm to (129.0, 70.0)
- moved U2 20.7 mm to (137.8, 77.4), turned to -90 degrees
- moved R3 16.6 mm to (145.8, 72.1), turned to 180 degrees
- moved U1 14.5 mm to (143.7, 56.8), turned to 180 degrees
- moved R4 12.6 mm to (141.2, 69.1), turned to -90 degrees
- moved U3 12.2 mm to (144.3, 79.8), turned to -90 degrees
- moved R2 11.0 mm to (121.3, 79.1), turned to -90 degrees
- moved C4 9.65 mm to (155.4, 91.2), turned to 90 degrees
- moved C2 8.37 mm to (136.1, 91.9)
- moved R5 3.42 mm to (152.4, 94.0), turned to 180 degrees
Connections:
- C3 pad 1: Net-(C1-Pad1) -> Net-(C3-Pad1)
- J2 pad 1: /SCL/A5 -> /SCL/A5*
- J2 pad 2: /SDA/A4 -> /SDA/A4*
- J3 pad 5: /SDA/A4 -> /SCL/A4
- J3 pad 6: /SCL/A5 -> /SDA/A5
- R3 pad 2: Net-(C1-Pad1) -> Net-(C3-Pad1)
- R4 pad 2: Net-(C1-Pad1) -> Net-(C3-Pad1)
- U2 pad 2: Net-(C1-Pad1) -> Net-(C3-Pad1)
- U4 pad 3: /A5 -> /SCL/A4
- U4 pad 4: /A4 -> /SDA/A5
Routing:
- net Net-(C3-Pad2): track 0.00 -> 130.5 mm, vias 0 -> 2
- net Net-(R1-Pad1): track 0.00 -> 55.2 mm
- net VCC: track 0.00 -> 50.7 mm
- net Net-(C1-Pad1): track 0.00 -> 28.0 mm
- net +5V: track 0.00 -> 25.4 mm
- net Net-(C3-Pad1): track 0.00 -> 22.1 mm
- net /SDA/A5: track 0.00 -> 18.3 mm
- net /SCL/A4: track 0.00 -> 17.9 mm
- net GND: track 0.00 -> 15.1 mm, vias 0 -> 2
- net /A0: track 0.00 -> 8.84 mm
- net /*11/RX: track 0.00 -> 8.75 mm
- net /*10/TX: track 0.00 -> 8.75 mm
- added copper zone on B.Cu, net GND
