File: KICAD/pcb_capteur_graphite_V2/pcb_capteur_graphite_V2.kicad_sch (KiCad schematic)
At the start: 16 parts, among them J1 Power, J2 Digital/PWM, J3 Analog, J4 Digital/PWM, U1 Blutooth_HC06, U2 LTC1050, U3 capteur

Commit message: Progression KICAD
Parts:
- added U4: oled, New_footprints:OLED, symbol New_symbols:oled
- C3: footprint (none) -> Capacitor_THT:C_Rect_L7.0mm_W4.5mm_P5.00mm
Connections:
- net *10/TX: now also U1.3 (TX); no longer U1. (VCC)
- net *11/RX: now also U1.4 (RX); no longer U1. (VCC)
- net A0: now also C4.1, R5.1
- net GND: now also U1.2 (GND), U4.2 (GND); no longer U1. (VCC)
- net VCC: now also U1.1 (VCC), U4.1 (VCC); no longer U1. (VCC)
- new net A4: U4.4 (SDA)
- new net A5: U4.3 (SCL)
Changed lines of the file:
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@@
   (junction (at 248.92 41.91) (diameter 0) (color 0 0 0 0)
+  )
+  (junction (at 270.51 49.53) (diameter 0) (color 0 0 0 0)
   )
   (junction (at 226.06 46.99) (diameter 0) (color 0 0 0 0)
@@
     (stroke (width 0) (type default) (color 0 0 0 0))
   )
+  (wire (pts (xy 219.71 83.82) (xy 219.71 92.71))
+    (stroke (width 0) (type default) (color 0 0 0 0))
+  )
   (wire (pts (xy 201.93 48.26) (xy 208.28 48.26))
     (stroke (width 0) (type default) (color 0 0 0 0))
@@
     (stroke (width 0) (type solid) (color 0 0 0 0))
   )
-  (wire (pts (xy 269.24 49.53) (xy 271.78 49.53))
+  (wire (pts (xy 269.24 49.53) (xy 270.51 49.53))
     (stroke (width 0) (type default) (color 0 0 0 0))
   )
@@
     (stroke (width 0) (type default) (color 0 0 0 0))
   )
+  (wire (pts (xy 275.59 45.72) (xy 270.51 45.72))
+    (stroke (width 0) (type default) (color 0 0 0 0))
+  )
   (wire (pts (xy 248.92 33.02) (xy 257.81 33.02))
     (stroke (width 0) (type default) (color 0 0 0 0))
@@
     (stroke (width 0) (type default) (color 0 0 0 0))
   )
+  (wire (pts (xy 212.09 83.82) (xy 212.09 92.71))
+    (stroke (width 0) (type default) (color 0 0 0 0))
+  )
   (polyline (pts (xy 280.67 16.51) (xy 280.67 68.58))
     (stroke (width 0) (type default) (color 0 0 0 0))
   )
+  (wire (pts (xy 217.17 83.82) (xy 217.17 92.71))
+    (stroke (width 0) (type default) (color 0 0 0 0))
+  )
   (wire (pts (xy 59.69 40.64) (xy 59.69 58.42))
     (stroke (width 0) (type solid) (color 0 0 0 0))
@@
     (stroke (width 0) (type solid) (color 0 0 0 0))
   )
+  (wire (pts (xy 270.51 45.72) (xy 270.51 49.53))
+    (stroke (width 0) (type default) (color 0 0 0 0))
+  )
   (wire (pts (xy 16.51 73.66) (xy 29.21 73.66))
     (stroke (width 0) (type solid) (color 0 0 0 0))
@@
     (stroke (width 0) (type default) (color 0 0 0 0))
   )
+  (wire (pts (xy 214.63 83.82) (xy 214.63 92.71))
+    (stroke (width 0) (type default) (color 0 0 0 0))
+  )
+  (wire (pts (xy 270.51 49.53) (xy 271.78 49.53))
+    (stroke (width 0) (type default) (color 0 0 0 0))
+  )
   (wire (pts (xy 218.44 31.75) (xy 240.03 31.75))
     (stroke (width 0) (type default) (color 0 0 0 0))
@@
     (effects (font (size 1.27 1.27)) (justify left bottom))
   )
+  (label "A5" (at 217.17 83.82 0)
+    (effects (font (size 1.27 1.27)) (justify left bottom))
+  )
   (label "VCC" (at 44.45 21.59 0)
     (effects (font (size 1.27 1.27)) (justify left bottom))
@@
     (effects (font (size 1.27 1.27)) (justify right bottom))
   )
+  (label "A0" (at 275.59 45.72 0)
+    (effects (font (size 1.27 1.27)) (justify left bottom))
+  )
   (label "2" (at 69.85 78.74 180)
     (effects (font (size 1.27 1.27)) (justify right bottom))
@@
     (effects (font (size 1.27 1.27)) (justify right bottom))
   )
+  (label "A4" (at 219.71 83.82 0)
+    (effects (font (size 1.27 1.27)) (justify left bottom))
+  )
   (label "*6" (at 69.85 68.58 180)
     (effects (font (size 1.27 1.27)) (justify right bottom))
@@
   )
   (label "IOREF" (at 13.97 40.64 0)
+    (effects (font (size 1.27 1.27)) (justify left bottom))
+  )
+  (label "VCC" (at 212.09 83.82 90)
     (effects (font (size 1.27 1.27)) (justify left bottom))
   )
@@
       (effects (font (size 1.27 1.27)) (justify left))
     )
-    (property "Footprint" "" (id 2) (at 249.8852 49.53 0)
+    (property "Footprint" "Capacitor_THT:C_Rect_L7.0mm_W4.5mm_P5.00mm" (id 2) (at 249.8852 49.53 0)
       (effects (font (size 1.27 1.27)) hide)
     )
@@
     (pin "1")
   )
+  (symbol (lib_name "GND_2") (lib_id "power:GND") (at 214.63 83.82 180) (unit 1)
+    (in_bom yes) (on_board yes) (fields_autoplaced)
+    (property "Reference" "#PWR0106" (id 0) (at 214.63 77.47 0)
+      (effects (font (size 1.27 1.27)) hide)
+    )
+    (property "Value" "GND" (id 1) (at 214.63 78.74 0))
+    (property "Footprint" "" (id 2) (at 214.63 83.82 0)
+      (effects (font (size 1.27 1.27)) hide)
+    )
+    (property "Datasheet" "" (id 3) (at 214.63 83.82 0)
+      (effects (font (size 1.27 1.27)) hide)
+    )
+    (pin "1")
+  )
   (symbol (lib_id "New_symbols:Blutooth_HC06") (at 168.91 88.9 0) (unit 1)
     (in_bom yes) (on_board yes)
@@
       (effects (font (size 1.27 1.27)) hide)
     )
-    (pin "")
-    (pin "")
-    (pin "")
-    (pin "")
+    (pin "1")
+    (pin "2")
+    (pin "3")
+    (pin "4")
   )
   (symbol (lib_id "power:PWR_FLAG") (at 31.75 19.05 0) (unit 1)
@@
     (pin "1")
     (pin "2")
+  )
+  (symbol (lib_id "New_symbols:oled") (at 199.39 87.63 0) (unit 1)
+    (in_bom yes) (on_board yes) (fields_autoplaced)
+    (property "Reference" "U4" (id 0) (at 223.52 95.2499 0)
+      (effects (font (size 1.27 1.27)) (justify left))
+    )
+    (property "Value" "oled" (id 1) (at 223.52 97.7899 0)
+      (effects (font (size 1.27 1.27)) (justify left))
+    )
+    (property "Footprint" "New_footprints:OLED" (id 2) (at 199.39 87.63 0)
+      (effects (font (size 1.27 1.27)) hide)
+    )
+    (property "Datasheet" "" (id 3) (at 199.39 87.63 0)
+      (effects (font (size 1.27 1.27)) hide)
+    )
+    (pin "1")
+    (pin "2")
+    (pin "3")
+    (pin "4")
   )
   (symbol (lib_id "power:VCC") (at 21.59 33.02 0) (unit 1)
@@
       (reference "#PWR0105") (unit 1) (value "+3.3V") (footprint "")
     )
+    (path "/3b113af7-3ec9-4b58-af47-d5b59fdc54e3"
+      (reference "#PWR0106") (unit 1) (value "GND") (footprint "")
+    )
     (path "/51caf9f4-e9f0-4b4a-a71c-590a0bf5400c"
       (reference "C1") (unit 1) (value "C") (footprint "Capacitor_THT:C_Disc_D3.0mm_W1.6mm_P2.50mm")
@@
     )
     (path "/1261c54b-782f-4308-99b5-9b6287a39cf3"
-      (reference "C3") (unit 1) (value "C") (footprint "")
+      (reference "C3") (unit 1) (value "C") (footprint "Capacitor_THT:C_Rect_L7.0mm_W4.5mm_P5.00mm")
     )
     (path "/ceaedd2f-69b3-4ee3-8ed8-c8b812f08c4c"
@@
       (reference "U3") (unit 1) (value "capteur") (footprint "New_footprints:capteur")
     )
-  )
+    (path "/59df8654-122d-457c-8e60-36e4f45bf3ee"
+      (reference "U4") (unit 1) (value "oled") (footprint "New_footprints:OLED")
+    )
+  )

Commit message: qq modification
Connections:
- net +5V: now also U2.7 (V+), U3.2 (IN); no longer U2. (V-), U3. (OUT)
- net GND: now also U2.4 (V-); no longer U2. (V-)
- net at C1.1, C3.1, R1.2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: now also U2.2 (IN-), U2.3 (IN+); no longer U2. (V-)
- net at C3.2, R4.1, R5.2: now also U2.6 (OUT); no longer U2. (V-)
- net at R1.1: now also U3.1 (OUT); no longer U3. (OUT)
Changed lines of the file:
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@@
   (junction (at 208.28 52.07) (diameter 0) (color 0 0 0 0)
   )
+  (junction (at 212.344 31.75) (diameter 0) (color 0 0 0 0)
+  )
   (junction (at 226.06 52.07) (diameter 0) (color 0 0 0 0)
   )
@@
   (junction (at 248.92 41.91) (diameter 0) (color 0 0 0 0)
   )
+  (junction (at 240.03 31.75) (diameter 0) (color 0 0 0 0)
+  )
   (junction (at 270.51 49.53) (diameter 0) (color 0 0 0 0)
   )
@@
   (junction (at 248.92 25.4) (diameter 0) (color 0 0 0 0)
   )
-  (junction (at 240.03 31.75) (diameter 0) (color 0 0 0 0)
+  (junction (at 220.98 31.75) (diameter 0) (color 0 0 0 0)
   )
   (junction (at 248.92 49.53) (diameter 0) (color 0 0 0 0)
@@
     (stroke (width 0) (type solid) (color 0 0 0 0))
   )
+  (wire (pts (xy 212.344 31.75) (xy 213.36 31.75))
+    (stroke (width 0) (type default) (color 0 0 0 0))
+  )
   (wire (pts (xy 57.15 73.66) (xy 69.85 73.66))
     (stroke (width 0) (type solid) (color 0 0 0 0))
@@
     (stroke (width 0) (type default) (color 0 0 0 0))
   )
-  (wire (pts (xy 240.03 31.75) (xy 240.03 25.4))
-    (stroke (width 0) (type default) (color 0 0 0 0))
-  )
   (wire (pts (xy 275.59 45.72) (xy 270.51 45.72))
     (stroke (width 0) (type default) (color 0 0 0 0))
@@
     (stroke (width 0) (type solid) (color 0 0 0 0))
   )
-  (wire (pts (xy 240.03 45.72) (xy 240.03 31.75))
+  (wire (pts (xy 240.03 25.4) (xy 240.03 31.75))
     (stroke (width 0) (type default) (color 0 0 0 0))
   )
@@
     (stroke (width 0) (type default) (color 0 0 0 0))
   )
-  (wire (pts (xy 213.36 31.75) (xy 194.31 31.75))
+  (wire (pts (xy 240.03 31.75) (xy 240.03 45.72))
+    (stroke (width 0) (type default) (color 0 0 0 0))
+  )
+  (wire (pts (xy 194.31 31.75) (xy 212.344 31.75))
     (stroke (width 0) (type default) (color 0 0 0 0))
   )
@@
     (stroke (width 0) (type default) (color 0 0 0 0))
   )
-  (wire (pts (xy 218.44 31.75) (xy 240.03 31.75))
+  (wire (pts (xy 218.44 31.75) (xy 220.98 31.75))
     (stroke (width 0) (type default) (color 0 0 0 0))
   )
@@
   (wire (pts (xy 57.15 76.2) (xy 69.85 76.2))
     (stroke (width 0) (type solid) (color 0 0 0 0))
+  )
+  (wire (pts (xy 220.98 31.75) (xy 240.03 31.75))
+    (stroke (width 0) (type default) (color 0 0 0 0))
   )
   (polyline (pts (xy 184.15 16.51) (xy 280.67 16.51))
@@
       (effects (font (size 1.27 1.27)) hide)
     )
-    (pin "")
-    (pin "")
-    (pin "")
-    (pin "")
-    (pin "")
+    (pin "2")
+    (pin "3")
+    (pin "4")
+    (pin "6")
+    (pin "7")
   )
   (symbol (lib_id "Device:C") (at 248.92 45.72 0) (unit 1)
@@
     (pin "2")
   )
-  (symbol (lib_id "New_symbols:capteur") (at 190.5 19.05 0) (unit 1)
-    (in_bom yes) (on_board yes) (fields_autoplaced)
-    (property "Reference" "U3" (id 0) (at 215.9 24.13 0))
-    (property "Value" "capteur" (id 1) (at 215.9 26.67 0))
-    (property "Footprint" "New_footprints:capteur" (id 2) (at 190.5 19.05 0)
-      (effects (font (size 1.27 1.27)) hide)
-    )
-    (property "Datasheet" "" (id 3) (at 190.5 19.05 0)
-      (effects (font (size 1.27 1.27)) hide)
-    )
-    (pin "")
-    (pin "")
+  (symbol (lib_id "New_symbols:capteur") (at 204.47 26.416 0) (unit 1)
+    (in_bom yes) (on_board yes) (fields_autoplaced)
+    (property "Reference" "U3" (id 0) (at 229.87 31.496 0))
+    (property "Value" "capteur" (id 1) (at 229.87 34.036 0))
+    (property "Footprint" "New_footprints:capteur" (id 2) (at 204.47 26.416 0)
+      (effects (font (size 1.27 1.27)) hide)
+    )
+    (property "Datasheet" "" (id 3) (at 204.47 26.416 0)
+      (effects (font (size 1.27 1.27)) hide)
+    )
+    (pin "1")
+    (pin "2")
   )
   (symbol (lib_id "power:+3V3") (at 55.88 21.59 270) (unit 1)

Commit message: le projet V2 le plus nouvelle dans session de yin, j'espere c'est le version qu'on a envoye au cathy
Parts:
- C1, C2, C4: footprint Capacitor_THT:C_Disc_D3.0mm_W1.6mm_P2.50mm -> New_footprints:Conductance
- R1, R2, R3, R4, R5: footprint Resistor_THT:R_Axial_DIN0204_L3.6mm_D1.6mm_P1.90mm_Vertical -> New_footprints:Resistor
Connections:
- net at C3.1, R3.2, R4.2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: no longer C1.1, R1.2, R2.2, U2.3 (IN+)
- net A4 renamed SDA/A5
- net SDA/A5: now also J3.6 (Pin_6)
- net A5 renamed SCL/A4
- net SCL/A4: now also J3.5 (Pin_5)
- net SCL/A5 renamed SCL/A5*
- net SCL/A5*: no longer J3.6 (Pin_6)
- net SDA/A4 renamed SDA/A4*
- net SDA/A4*: no longer J3.5 (Pin_5)
- new net: C1.1, R1.2, R2.2, U2.3 (IN+)
